Commit message: fix: urdf

File: tutorial/01 - models/data/GenericDH_6dof_11.urdf (robot description, URDF)
Before this commit: robot GenericDH, 12 links, 11 joints
Joints:
- joint move_l4_from_a4: axis 0.0 -1.2246467991473532e-16 -1.0 -> 0.0 0 -1.0

Commit message: fix: urdf

File: tutorial/01 - models/data/GenericDH_6dof_11.urdf (robot description, URDF)
Before this commit: robot GenericDH, 12 links, 11 joints
Joints:
- joint move_l4_from_a4: axis 0.0 0 -1.0 -> 0.0 -1.2246467991473532e-16 -1.0
